File: extron-input/scart-input.kicad_pcb (KiCad board)
At the start: 2 copper layers, 92 x 37 mm, 16 parts, among them J1 SCART-F, J10 Conn_01x01, J11 Conn_01x01, J2 RED, J3 GREEN, J4 BLUE, J5 SYNC, J6 PHOENIX, J7 SENSE, J8 SENSE, J9 Conn_01x01, SW1 SW_DPDT_x2, U1 LM1881

Commit message: Rename things to scart-input
Parts:
- J1: footprint extron-scart:SCART_F_RA -> scart-input:SCART_F_RA
- J2, J3, J4, J5: footprint extron-scart:BNC_90 -> scart-input:BNC_90
Changed lines of the file:
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@@
     )
   )
-  (module extron-scart:BNC_90 (layer F.Cu)
+  (module scart-input:BNC_90 (layer F.Cu)
     (at 152.4 76.2 180)
     (descr "BNC connector, Tyco 1-1337543-0")
@@
     )
   )
-  (module extron-scart:BNC_90 (layer F.Cu)
+  (module scart-input:BNC_90 (layer F.Cu)
     (at 132.08 76.2 180)
     (descr "BNC connector, Tyco 1-1337543-0")
@@
     )
   )
-  (module extron-scart:BNC_90 (layer F.Cu)
+  (module scart-input:BNC_90 (layer F.Cu)
     (at 111.76 76.2 180)
     (descr "BNC connector, Tyco 1-1337543-0")
@@
     )
   )
-  (module extron-scart:BNC_90 (layer F.Cu)
+  (module scart-input:BNC_90 (layer F.Cu)
     (at 91.44 76.2 180)
     (descr "BNC connector, Tyco 1-1337543-0")
@@
     )
   )
-  (module extron-scart:SCART_F_RA (layer F.Cu)
+  (module scart-input:SCART_F_RA (layer F.Cu)
     (at 129.921 104.9655 180)
     (fp_text reference J1 (at 0.1778 -4.4577 180) (layer F.SilkS)
