File: extron-input/scart-input.sch (KiCad schematic (older format))
At the start: 16 parts, among them J1 SCART-F, J10 Conn_01x01, J11 Conn_01x01, J2 Conn_Coaxial, J3 Conn_Coaxial, J4 Conn_Coaxial, J5 Conn_Coaxial, J6 Conn_01x03_Male, J7 Conn_01x02_Male, J8 Conn_01x01, J9 Conn_01x01, SW1 SW_DPDT_x2, U1 LM1881

Commit message: Rename things to scart-input
Parts:
- J1: footprint extron-scart:SCART_F_RA -> scart-input:SCART_F_RA
- J2, J3, J4, J5: footprint extron-scart:BNC_90 -> scart-input:BNC_90
Changed lines of the file:
@@
 LIBS:power
 LIBS:74xx
-LIBS:extron-scart-cache
+LIBS:scart-input-cache
 EELAYER 26 0
 EELAYER END
@@
 F 0 "J2" H 8200 1550 50  0000 L CNN
 F 1 "Conn_Coaxial" H 7850 2200 50  0000 L CNN
-F 2 "extron-scart:BNC_90" H 8250 2050 50  0001 C CNN
+F 2 "scart-input:BNC_90" H 8250 2050 50  0001 C CNN
 F 3 " ~" H 8250 2050 50  0001 C CNN
 	1    8250 2050
@@
 F 0 "J3" H 8200 2400 50  0000 L CNN
 F 1 "Conn_Coaxial" H 7850 3050 50  0000 L CNN
-F 2 "extron-scart:BNC_90" H 8250 2900 50  0001 C CNN
+F 2 "scart-input:BNC_90" H 8250 2900 50  0001 C CNN
 F 3 " ~" H 8250 2900 50  0001 C CNN
 	1    8250 2900
@@
 F 0 "J4" H 8200 3250 50  0000 L CNN
 F 1 "Conn_Coaxial" H 7850 3900 50  0000 L CNN
-F 2 "extron-scart:BNC_90" H 8250 3750 50  0001 C CNN
+F 2 "scart-input:BNC_90" H 8250 3750 50  0001 C CNN
 F 3 " ~" H 8250 3750 50  0001 C CNN
 	1    8250 3750
@@
 F 0 "J5" H 8200 4050 50  0000 L CNN
 F 1 "Conn_Coaxial" H 7850 4700 50  0000 L CNN
-F 2 "extron-scart:BNC_90" H 8250 4550 50  0001 C CNN
+F 2 "scart-input:BNC_90" H 8250 4550 50  0001 C CNN
 F 3 " ~" H 8250 4550 50  0001 C CNN
 	1    8250 4550
@@
 F 0 "J1" H 3850 4520 50  0000 C CNN
 F 1 "SCART-F" H 3850 4429 50  0000 C CNN
-F 2 "extron-scart:SCART_F_RA" H 3850 3150 50  0001 C CNN
+F 2 "scart-input:SCART_F_RA" H 3850 3150 50  0001 C CNN
 F 3 " ~" H 3850 3150 50  0001 C CNN
 	1    3850 3100
