File: extron-input/extron-input.sch (KiCad schematic (older format))
At the start: 24 parts, among them J1 SCART-F, J10 Conn_01x01, J11 Conn_01x01, J12 RED, J13 GREEN, J14 BLUE, J15 SYNC, J2 RED, J3 GREEN, J4 BLUE, J5 SYNC, J6 PHOENIX, J7 SENSE, J8 Conn_01x01, J9 Conn_01x01, SW1 SW_DPDT_x2, U1 LM1881

Commit message: Rev 2.1
Fixed up rca problems by making combined footprint for the two different
CUI-style connectors.
Shifted scart over so it doesn't run into standoffs (hopefully)
Fixed resistor value in sense circuit
Reversed stereo audio signals
Added logos + link to site
Parts:
- removed J12: RED, extron-input:rca_black, symbol Connector:Conn_Coaxial
- removed J13: GREEN, extron-input:rca_black, symbol Connector:Conn_Coaxial
- removed J14: BLUE, extron-input:rca_black, symbol Connector:Conn_Coaxial
- removed J15: SYNC, extron-input:rca_black, symbol Connector:Conn_Coaxial
- C1, C2: symbol Device:C_Small -> extron-input-rescue:C_Small-Device
- D1: symbol Device:D_ALT -> extron-input-rescue:D_ALT-Device
- D2: symbol Device:D_Zener -> extron-input-rescue:D_Zener-Device
- J1: symbol Connector:SCART-F -> extron-input-rescue:SCART-F-Connector
- J10, J11, J8, J9: symbol Connector_Generic:Conn_01x01 -> extron-input-rescue:Conn_01x01-Connector_Generic
- J2, J3, J4, J5: footprint extron-input:rca_boom -> extron-input:rca_combined; symbol Connector:Conn_Coaxial -> extron-input-rescue:Conn_Coaxial-Connector
- J6: symbol Connector:Conn_01x03_Male -> extron-input-rescue:Conn_01x03_Male-Connector
- J7: symbol Connector:Conn_01x02_Male -> extron-input-rescue:Conn_01x02_Male-Connector
- R1, R3: symbol Device:R_US -> extron-input-rescue:R_US-Device
- R2: value 100KΩ -> 100Ω; symbol Device:R_US -> extron-input-rescue:R_US-Device
- SW1: symbol Switch:SW_DPDT_x2 -> extron-input-rescue:SW_DPDT_x2-Switch
- U1: symbol Video:LM1881 -> extron-input-rescue:LM1881-Video
Connections:
- net BLUE: now also J4.2 (Ext); no longer J4.1 (In)
- net GND: now also J2.1 (In), J3.1 (In), J4.1 (In), J5.1 (In); no longer J2.2 (Ext), J3.2 (Ext), J4.2 (Ext), J5.2 (Ext)
- net GREEN: now also J3.2 (Ext); no longer J3.1 (In)
- net RED: now also J2.2 (Ext); no longer J2.1 (In)
- net SYNC: now also J5.2 (Ext); no longer J5.1 (In)
- net at J1.2 (P2): now also J6.3 (Pin_3); no longer J6.1 (Pin_1)
- net at J1.6 (P6): now also J6.1 (Pin_1); no longer J6.3 (Pin_3)
Other:
- moved on the sheet: J6
Changed lines of the file:
@@
 LIBS:74xx
 LIBS:extron-input-cache
-EELAYER 26 0
+EELAYER 29 0
 EELAYER END
 $Descr A4 11693 8268
 encoding utf-8
 Sheet 1 1
-Title ""
-Date ""
-Rev ""
-Comp ""
+Title "Extron Scart Adapter (Input)"
+Date "2019-03-28"
+Rev "2.1"
+Comp "Rattboi (Bradon Kanyid)"
 Comment1 ""
 Comment2 ""
@@
 BLUE
 NoConn ~ 4450 2600
+Text GLabel 8050 2050 0    60   Input ~ 0
+GND
+Text GLabel 8250 4750 3    60   Input ~ 0
+SYNC
+Text GLabel 8250 3100 3    60   Input ~ 0
+GREEN
+Text GLabel 8250 3950 3    60   Input ~ 0
+BLUE
 Text GLabel 8250 2250 3    60   Input ~ 0
+RED
+Text GLabel 8050 2900 0    60   Input ~ 0
+GND
+Text GLabel 8050 3750 0    60   Input ~ 0
 GND
 Text GLabel 8050 4550 0    60   Input ~ 0
-SYNC
-Text GLabel 8050 2900 0    60   Input ~ 0
-GREEN
-Text GLabel 8050 3750 0    60   Input ~ 0
-BLUE
-Text GLabel 8050 2050 0    60   Input ~ 0
-RED
-Text GLabel 8250 3100 3    60   Input ~ 0
-GND
-Text GLabel 8250 3950 3    60   Input ~ 0
-GND
-Text GLabel 8250 4750 3    60   Input ~ 0
-GND
-$Comp
-L Connector:SCART-F J1
+GND
+$Comp
+L extron-input-rescue:SCART-F-Connector J1
 U 1 1 5C652397
 P 3850 3100
@@
 $EndComp
 $Comp
-L Connector:Conn_01x03_Male J6
+L extron-input-rescue:Conn_01x03_Male-Connector J6
 U 1 1 5C652866
-P 4650 4550
-F 0 "J6" H 4756 4828 50  0000 C CNN
-F 1 "PHOENIX" H 4756 4737 50  0000 C CNN
-F 2 "Connector_JST:JST_XH_S03B-XH-A_1x03_P2.50mm_Horizontal" H 4650 4550 50  0001 C CNN
-F 3 "~" H 4650 4550 50  0001 C CNN
-F 4 "https://lcsc.com/product-detail/XH-Connectors_JST_S3B-XH-A-LF-SN_XHsocket-1-3P-Curved-needle-pitch2-5mm_C157928.html" H 4650 4550 50  0001 C CNN "Vendor"
-	1    4650 4550
-	1    0    0    -1
-$EndComp
-$Comp
-L Connector:Conn_01x02_Male J7
+P 4650 4750
+F 0 "J6" H 4756 5028 50  0000 C CNN
+F 1 "PHOENIX" H 4756 4937 50  0000 C CNN
+F 2 "Connector_JST:JST_XH_S03B-XH-A_1x03_P2.50mm_Horizontal" H 4650 4750 50  0001 C CNN
+F 3 "~" H 4650 4750 50  0001 C CNN
+F 4 "https://lcsc.com/product-detail/XH-Connectors_JST_S3B-XH-A-LF-SN_XHsocket-1-3P-Curved-needle-pitch2-5mm_C157928.html" H 4650 4750 50  0001 C CNN "Vendor"
+	1    4650 4750
+	1    0    0    -1
+$EndComp
+$Comp
+L extron-input-rescue:Conn_01x02_Male-Connector J7
 U 1 1 5C74DAFA
 P 5750 5800
@@
 $EndComp
 $Comp
-L Video:LM1881 U1
+L extron-input-rescue:LM1881-Video U1
 U 1 1 5C74DDC8
 P 6750 2400
@@
 $EndComp
 $Comp
-L Device:R_US R1
+L extron-input-rescue:R_US-Device R1
 U 1 1 5C74E55F
 P 5800 2850
@@
 $EndComp
 $Comp
-L Device:C_Small C2
+L extron-input-rescue:C_Small-Device C2
 U 1 1 5C74EC46
 P 5800 2500
@@
 	6000 2500 6200 2500
 $Comp
-L power:GND #PWR0101
+L extron-input-rescue:GND-power #PWR0101
 U 1 1 5C74F12A
 P 5450 2550
@@
 	6200 2400 6250 2400
 $Comp
-L Device:C_Small C1
+L extron-input-rescue:C_Small-Device C1
 U 1 1 5C74F422
 P 5800 2300
@@
 	5900 2300 6250 2300
 $Comp
-L power:GND #PWR0102
+L extron-input-rescue:GND-power #PWR0102
 U 1 1 5C74FB45
 P 6750 2700
@@
 $EndComp
 $Comp
-L Switch:SW_DPDT_x2 SW1
+L extron-input-rescue:SW_DPDT_x2-Switch SW1
 U 2 1 5C75001B
 P 5100 3400
@@
 $EndComp
 $Comp
-L Switch:SW_DPDT_x2 SW1
+L extron-input-rescue:SW_DPDT_x2-Switch SW1
 U 1 1 5C7500A7
 P 5050 2200
@@
 Wire Wire Line
 	4450 3800 5250 3800
-Wire Wire Line
-	5250 4550 4850 4550
-Wire Wire Line
-	5250 3800 5250 4550
 Text GLabel 4450 2800 2    50   Input ~ 0
 GND
@@
 NoConn ~ 2400 6200
 $Comp
-L Connector_Generic:Conn_01x01 J8
+L extron-input-rescue:Conn_01x01-Connector_Generic J8
 U 1 1 5C7605B3
 P 2600 5600
@@
 $EndComp
 $Comp
-L Connector_Generic:Conn_01x01 J9
+L extron-input-rescue:Conn_01x01-Connector_Generic J9
 U 1 1 5C76074F
 P 2600 5800
@@
 $EndComp
 $Comp
-L Connector_Generic:Conn_01x01 J10
+L extron-input-rescue:Conn_01x01-Connector_Generic J10
 U 1 1 5C760785
 P 2600 6000
@@
 $EndComp
 $Comp
-L Connector_Generic:Conn_01x01 J11
+L extron-input-rescue:Conn_01x01-Connector_Generic J11
 U 1 1 5C7607B9
 P 2600 6200
@@
 	4450 4000 5050 4000
 Wire Wire Line
-	5050 4000 5050 4450
-Wire Wire Line
-	5050 4450 4850 4450
-Wire Wire Line
 	5450 3600 5450 4650
 Wire Wire Line
@@
 	5550 5700 5500 5700
 $Comp
-L Device:D_ALT D1
+L extron-input-rescue:D_ALT-Device D1
 U 1 1 5C84733C
 P 4350 5700
@@
 $EndComp
 $Comp
-L Device:R_US R2
+L extron-input-rescue:R_US-Device R2
 U 1 1 5C847B71
 P 4800 5700
 F 0 "R2" V 4595 5700 50  0000 C CNN
-F 1 "100KΩ" V 4686 5700 50  0000 C CNN
+F 1 "100Ω" V 4686 5700 50  0000 C CNN
 F 2 "Resistor_THT:R_Axial_DIN0204_L3.6mm_D1.6mm_P1.90mm_Vertical" V 4840 5690 50  0001 C CNN
 F 3 "~" H 4800 5700 50  0001 C CNN
@@
 $EndComp
 $Comp
-L Device:D_Zener D2
+L extron-input-rescue:D_Zener-Device D2
 U 1 1 5C847C9D
 P 5050 5850
@@
 SENSE
 $Comp
-L power:GND #PWR0103
+L extron-input-rescue:GND-power #PWR0103
 U 1 1 5C849937
 P 5050 6050
@@
 	5050 6000 5050 6050
 $Comp
-L Device:R_US R3
+L extron-input-rescue:R_US-Device R3
 U 1 1 5C84AF3E
 P 5350 5700
@@
 	4500 5700 4650 5700
 $Comp
-L Connector:Conn_Coaxial J12
-U 1 1 5C84CB4A
-P 8650 2050
-F 0 "J12" H 8750 2026 50  0000 L CNN
-F 1 "RED" H 8750 1935 50  0000 L CNN
-F 2 "extron-input:rca_black" H 8650 2050 50  0001 C CNN
-F 3 " ~" H 8650 2050 50  0001 C CNN
-F 4 "https://www.arrow.com/en/products/rcj-042/cui-inc" H 8650 2050 50  0001 C CNN "Vendor"
-	1    8650 2050
-	1    0    0    -1
-$EndComp
-Wire Wire Line
-	8050 1850 8050 2050
-Wire Wire Line
-	8250 2250 8650 2250
-Wire Wire Line
-	8050 1850 8450 1850
-Wire Wire Line
-	8450 1850 8450 2050
-$Comp
-L Connector:Conn_Coaxial J13
-U 1 1 5C84FDFD
-P 8650 2900
-F 0 "J13" H 8750 2876 50  0000 L CNN
-F 1 "GREEN" H 8750 2785 50  0000 L CNN
-F 2 "extron-input:rca_black" H 8650 2900 50  0001 C CNN
-F 3 " ~" H 8650 2900 50  0001 C CNN
-F 4 "https://www.arrow.com/en/products/rcj-046/cui-inc" H 8650 2900 50  0001 C CNN "Vendor"
-	1    8650 2900
-	1    0    0    -1
-$EndComp
-$Comp
-L Connector:Conn_Coaxial J14
-U 1 1 5C84FE72
-P 8650 3750
-F 0 "J14" H 8749 3726 50  0000 L CNN
-F 1 "BLUE" H 8749 3635 50  0000 L CNN
-F 2 "extron-input:rca_black" H 8650 3750 50  0001 C CNN
-F 3 " ~" H 8650 3750 50  0001 C CNN
-F 4 "https://www.arrow.com/en/products/rcj-045/cui-inc" H 8650 3750 50  0001 C CNN "Vendor"
-	1    8650 3750
-	1    0    0    -1
-$EndComp
-$Comp
-L Connector:Conn_Coaxial J15
-U 1 1 5C84FF62
-P 8650 4550
-F 0 "J15" H 8750 4526 50  0000 L CNN
-F 1 "SYNC" H 8750 4435 50  0000 L CNN
-F 2 "extron-input:rca_black" H 8650 4550 50  0001 C CNN
-F 3 " ~" H 8650 4550 50  0001 C CNN
-F 4 "https://www.arrow.com/en/products/rcj-044/cui-inc" H 8650 4550 50  0001 C CNN "Vendor"
-	1    8650 4550
-	1    0    0    -1
-$EndComp
-Wire Wire Line
-	8650 4750 8250 4750
-Wire Wire Line
-	8450 4550 8450 4400
-Wire Wire Line
-	8450 4400 8050 4400
-Wire Wire Line
-	8050 4400 8050 4550
-Wire Wire Line
-	8650 3950 8250 3950
-Wire Wire Line
-	8050 3750 8050 3600
-Wire Wire Line
-	8050 3600 8450 3600
-Wire Wire Line
-	8450 3600 8450 3750
-Wire Wire Line
-	8250 3100 8650 3100
-Wire Wire Line
-	8050 2900 8050 2750
-Wire Wire Line
-	8050 2750 8450 2750
-Wire Wire Line
-	8450 2750 8450 2900
-$Comp
-L Connector:Conn_Coaxial J2
+L extron-input-rescue:Conn_Coaxial-Connector J2
 U 1 1 5C8498CA
 P 8250 2050
 F 0 "J2" H 8350 2026 50  0000 L CNN
 F 1 "RED" H 8350 1935 50  0000 L CNN
-F 2 "extron-input:rca_boom" H 8250 2050 50  0001 C CNN
+F 2 "extron-input:rca_combined" H 8250 2050 50  0001 C CNN
 F 3 " ~" H 8250 2050 50  0001 C CNN
 F 4 "https://lcsc.com/product-detail/AV-Connectors_AV-5_C18080.html" H 8250 2050 50  0001 C CNN "Vendor"
@@
 $EndComp
 $Comp
-L Connector:Conn_Coaxial J3
+L extron-input-rescue:Conn_Coaxial-Connector J3
 U 1 1 5C849928
 P 8250 2900
 F 0 "J3" H 8350 2876 50  0000 L CNN
 F 1 "GREEN" H 8350 2785 50  0000 L CNN
-F 2 "extron-input:rca_boom" H 8250 2900 50  0001 C CNN
+F 2 "extron-input:rca_combined" H 8250 2900 50  0001 C CNN
 F 3 " ~" H 8250 2900 50  0001 C CNN
 F 4 "https://lcsc.com/product-detail/AV-Connectors_AV-5_C18080.html" H 8250 2900 50  0001 C CNN "Vendor"
@@
 $EndComp
 $Comp
-L Connector:Conn_Coaxial J4
+L extron-input-rescue:Conn_Coaxial-Connector J4
 U 1 1 5C84997A
 P 8250 3750
 F 0 "J4" H 8349 3726 50  0000 L CNN
 F 1 "BLUE" H 8349 3635 50  0000 L CNN
-F 2 "extron-input:rca_boom" H 8250 3750 50  0001 C CNN
+F 2 "extron-input:rca_combined" H 8250 3750 50  0001 C CNN
 F 3 " ~" H 8250 3750 50  0001 C CNN
 F 4 "https://lcsc.com/product-detail/AV-Connectors_AV-5_C18080.html" H 8250 3750 50  0001 C CNN "Vendor"
@@
 $EndComp
 $Comp
-L Connector:Conn_Coaxial J5
+L extron-input-rescue:Conn_Coaxial-Connector J5
 U 1 1 5C8499F8
 P 8250 4550
 F 0 "J5" H 8350 4526 50  0000 L CNN
 F 1 "SYNC" H 8350 4435 50  0000 L CNN
-F 2 "extron-input:rca_boom" H 8250 4550 50  0001 C CNN
+F 2 "extron-input:rca_combined" H 8250 4550 50  0001 C CNN
 F 3 " ~" H 8250 4550 50  0001 C CNN
 F 4 "https://lcsc.com/product-detail/AV-Connectors_AV-5_C18080.html" H 8250 4550 50  0001 C CNN "Vendor"
@@
 	1    0    0    -1
 $EndComp
+Wire Wire Line
+	5050 4850 4850 4850
+Wire Wire Line
+	5050 4000 5050 4850
+Wire Wire Line
+	5250 4750 4850 4750
+Wire Wire Line
+	5250 3800 5250 4750
 $EndSCHEMATC

Commit message: Update extron output board to use combined RCA (v2.1)
Small fixes for extron input as well (v2.1)
Parts:
- C1, C2: symbol extron-input-rescue:C_Small-Device -> extron-input-rescue:C_Small-Device-extron-input-rescue
- D1: symbol extron-input-rescue:D_ALT-Device -> extron-input-rescue:D_ALT-Device-extron-input-rescue
- D2: symbol extron-input-rescue:D_Zener-Device -> extron-input-rescue:D_Zener-Device-extron-input-rescue
- J1: symbol extron-input-rescue:SCART-F-Connector -> extron-input-rescue:SCART-F-Connector-extron-input-rescue
- J10, J11, J8, J9: symbol extron-input-rescue:Conn_01x01-Connector_Generic -> extron-input-rescue:Conn_01x01-Connector_Generic-extron-input-rescue
- J2, J3, J4, J5: symbol extron-input-rescue:Conn_Coaxial-Connector -> extron-input-rescue:Conn_Coaxial-Connector-extron-input-rescue
- J6: symbol extron-input-rescue:Conn_01x03_Male-Connector -> extron-input-rescue:Conn_01x03_Male-Connector-extron-input-rescue
- J7: symbol extron-input-rescue:Conn_01x02_Male-Connector -> extron-input-rescue:Conn_01x02_Male-Connector-extron-input-rescue
- R1, R2, R3: symbol extron-input-rescue:R_US-Device -> extron-input-rescue:R_US-Device-extron-input-rescue
- SW1: symbol extron-input-rescue:SW_DPDT_x2-Switch -> extron-input-rescue:SW_DPDT_x2-Switch-extron-input-rescue
- U1: symbol extron-input-rescue:LM1881-Video -> extron-input-rescue:LM1881-Video-extron-input-rescue
Changed lines of the file:
@@
 GND
 $Comp
-L extron-input-rescue:SCART-F-Connector J1
+L extron-input-rescue:SCART-F-Connector-extron-input-rescue J1
 U 1 1 5C652397
 P 3850 3100
@@
 $EndComp
 $Comp
-L extron-input-rescue:Conn_01x03_Male-Connector J6
+L extron-input-rescue:Conn_01x03_Male-Connector-extron-input-rescue J6
 U 1 1 5C652866
 P 4650 4750
@@
 $EndComp
 $Comp
-L extron-input-rescue:Conn_01x02_Male-Connector J7
+L extron-input-rescue:Conn_01x02_Male-Connector-extron-input-rescue J7
 U 1 1 5C74DAFA
 P 5750 5800
@@
 $EndComp
 $Comp
-L extron-input-rescue:LM1881-Video U1
+L extron-input-rescue:LM1881-Video-extron-input-rescue U1
 U 1 1 5C74DDC8
 P 6750 2400
@@
 $EndComp
 $Comp
-L extron-input-rescue:R_US-Device R1
+L extron-input-rescue:R_US-Device-extron-input-rescue R1
 U 1 1 5C74E55F
 P 5800 2850
@@
 $EndComp
 $Comp
-L extron-input-rescue:C_Small-Device C2
+L extron-input-rescue:C_Small-Device-extron-input-rescue C2
 U 1 1 5C74EC46
 P 5800 2500
@@
 	6000 2500 6200 2500
 $Comp
-L extron-input-rescue:GND-power #PWR0101
+L extron-input-rescue:GND-power-extron-input-rescue #PWR0101
 U 1 1 5C74F12A
 P 5450 2550
@@
 	6200 2400 6250 2400
 $Comp
-L extron-input-rescue:C_Small-Device C1
+L extron-input-rescue:C_Small-Device-extron-input-rescue C1
 U 1 1 5C74F422
 P 5800 2300
@@
 	5900 2300 6250 2300
 $Comp
-L extron-input-rescue:GND-power #PWR0102
+L extron-input-rescue:GND-power-extron-input-rescue #PWR0102
 U 1 1 5C74FB45
 P 6750 2700
@@
 $EndComp
 $Comp
-L extron-input-rescue:SW_DPDT_x2-Switch SW1
+L extron-input-rescue:SW_DPDT_x2-Switch-extron-input-rescue SW1
 U 2 1 5C75001B
 P 5100 3400
@@
 $EndComp
 $Comp
-L extron-input-rescue:SW_DPDT_x2-Switch SW1
+L extron-input-rescue:SW_DPDT_x2-Switch-extron-input-rescue SW1
 U 1 1 5C7500A7
 P 5050 2200
@@
 NoConn ~ 2400 6200
 $Comp
-L extron-input-rescue:Conn_01x01-Connector_Generic J8
+L extron-input-rescue:Conn_01x01-Connector_Generic-extron-input-rescue J8
 U 1 1 5C7605B3
 P 2600 5600
@@
 $EndComp
 $Comp
-L extron-input-rescue:Conn_01x01-Connector_Generic J9
+L extron-input-rescue:Conn_01x01-Connector_Generic-extron-input-rescue J9
 U 1 1 5C76074F
 P 2600 5800
@@
 $EndComp
 $Comp
-L extron-input-rescue:Conn_01x01-Connector_Generic J10
+L extron-input-rescue:Conn_01x01-Connector_Generic-extron-input-rescue J10
 U 1 1 5C760785
 P 2600 6000
@@
 $EndComp
 $Comp
-L extron-input-rescue:Conn_01x01-Connector_Generic J11
+L extron-input-rescue:Conn_01x01-Connector_Generic-extron-input-rescue J11
 U 1 1 5C7607B9
 P 2600 6200
@@
 	5550 5700 5500 5700
 $Comp
-L extron-input-rescue:D_ALT-Device D1
+L extron-input-rescue:D_ALT-Device-extron-input-rescue D1
 U 1 1 5C84733C
 P 4350 5700
@@
 $EndComp
 $Comp
-L extron-input-rescue:R_US-Device R2
+L extron-input-rescue:R_US-Device-extron-input-rescue R2
 U 1 1 5C847B71
 P 4800 5700
@@
 $EndComp
 $Comp
-L extron-input-rescue:D_Zener-Device D2
+L extron-input-rescue:D_Zener-Device-extron-input-rescue D2
 U 1 1 5C847C9D
 P 5050 5850
@@
 SENSE
 $Comp
-L extron-input-rescue:GND-power #PWR0103
+L extron-input-rescue:GND-power-extron-input-rescue #PWR0103
 U 1 1 5C849937
 P 5050 6050
@@
 	5050 6000 5050 6050
 $Comp
-L extron-input-rescue:R_US-Device R3
+L extron-input-rescue:R_US-Device-extron-input-rescue R3
 U 1 1 5C84AF3E
 P 5350 5700
@@
 	4500 5700 4650 5700
 $Comp
-L extron-input-rescue:Conn_Coaxial-Connector J2
+L extron-input-rescue:Conn_Coaxial-Connector-extron-input-rescue J2
 U 1 1 5C8498CA
 P 8250 2050
@@
 $EndComp
 $Comp
-L extron-input-rescue:Conn_Coaxial-Connector J3
+L extron-input-rescue:Conn_Coaxial-Connector-extron-input-rescue J3
 U 1 1 5C849928
 P 8250 2900
@@
 $EndComp
 $Comp
-L extron-input-rescue:Conn_Coaxial-Connector J4
+L extron-input-rescue:Conn_Coaxial-Connector-extron-input-rescue J4
 U 1 1 5C84997A
 P 8250 3750
@@
 $EndComp
 $Comp
-L extron-input-rescue:Conn_Coaxial-Connector J5
+L extron-input-rescue:Conn_Coaxial-Connector-extron-input-rescue J5
 U 1 1 5C8499F8
 P 8250 4550
