File: extron-input/extron-input.sch (KiCad schematic (older format))
At the start: 20 parts, among them J1 SCART-F, J10 Conn_01x01, J11 Conn_01x01, J2 RED, J3 GREEN, J4 BLUE, J5 SYNC, J6 PHOENIX, J7 SENSE, J8 Conn_01x01, J9 Conn_01x01, SW1 SW_DPDT_x2, U1 LM1881

Commit message: Add mounting holes and 2nd position for serial uart on switchboard
Also, "rescue" components on scart-input board. I gotta figure out what
that's about...
Parts:
- C1, C2: symbol extron-input-rescue:C_Small-Device-extron-input-rescue -> extron-input-rescue:C_Small-Device-extron-input-rescue-extron-input-rescue
- D1: symbol extron-input-rescue:D_ALT-Device-extron-input-rescue -> extron-input-rescue:D_ALT-Device-extron-input-rescue-extron-input-rescue
- D2: symbol extron-input-rescue:D_Zener-Device-extron-input-rescue -> extron-input-rescue:D_Zener-Device-extron-input-rescue-extron-input-rescue
- J1: symbol extron-input-rescue:SCART-F-Connector-extron-input-rescue -> extron-input-rescue:SCART-F-Connector-extron-input-rescue-extron-input-rescue
- J10, J11, J8, J9: symbol extron-input-rescue:Conn_01x01-Connector_Generic-extron-input-rescue -> extron-input-rescue:Conn_01x01-Connector_Generic-extron-input-rescue-extron-input-rescue
- J2, J3, J4, J5: symbol extron-input-rescue:Conn_Coaxial-Connector-extron-input-rescue -> extron-input-rescue:Conn_Coaxial-Connector-extron-input-rescue-extron-input-rescue
- J6: symbol extron-input-rescue:Conn_01x03_Male-Connector-extron-input-rescue -> extron-input-rescue:Conn_01x03_Male-Connector-extron-input-rescue-extron-input-rescue
- J7: symbol extron-input-rescue:Conn_01x02_Male-Connector-extron-input-rescue -> extron-input-rescue:Conn_01x02_Male-Connector-extron-input-rescue-extron-input-rescue
- R1, R2, R3: symbol extron-input-rescue:R_US-Device-extron-input-rescue -> extron-input-rescue:R_US-Device-extron-input-rescue-extron-input-rescue
- SW1: symbol extron-input-rescue:SW_DPDT_x2-Switch-extron-input-rescue -> extron-input-rescue:SW_DPDT_x2-Switch-extron-input-rescue-extron-input-rescue
- U1: symbol extron-input-rescue:LM1881-Video-extron-input-rescue -> extron-input-rescue:LM1881-Video-extron-input-rescue-extron-input-rescue
Changed lines of the file:
@@
 GND
 $Comp
-L extron-input-rescue:SCART-F-Connector-extron-input-rescue J1
+L extron-input-rescue:SCART-F-Connector-extron-input-rescue-extron-input-rescue J1
 U 1 1 5C652397
 P 3850 3100
@@
 $EndComp
 $Comp
-L extron-input-rescue:Conn_01x03_Male-Connector-extron-input-rescue J6
+L extron-input-rescue:Conn_01x03_Male-Connector-extron-input-rescue-extron-input-rescue J6
 U 1 1 5C652866
 P 4650 4750
@@
 $EndComp
 $Comp
-L extron-input-rescue:Conn_01x02_Male-Connector-extron-input-rescue J7
+L extron-input-rescue:Conn_01x02_Male-Connector-extron-input-rescue-extron-input-rescue J7
 U 1 1 5C74DAFA
 P 5750 5800
@@
 $EndComp
 $Comp
-L extron-input-rescue:LM1881-Video-extron-input-rescue U1
+L extron-input-rescue:LM1881-Video-extron-input-rescue-extron-input-rescue U1
 U 1 1 5C74DDC8
 P 6750 2400
@@
 $EndComp
 $Comp
-L extron-input-rescue:R_US-Device-extron-input-rescue R1
+L extron-input-rescue:R_US-Device-extron-input-rescue-extron-input-rescue R1
 U 1 1 5C74E55F
 P 5800 2850
@@
 $EndComp
 $Comp
-L extron-input-rescue:C_Small-Device-extron-input-rescue C2
+L extron-input-rescue:C_Small-Device-extron-input-rescue-extron-input-rescue C2
 U 1 1 5C74EC46
 P 5800 2500
@@
 	6000 2500 6200 2500
 $Comp
-L extron-input-rescue:GND-power-extron-input-rescue #PWR0101
+L extron-input-rescue:GND-power-extron-input-rescue-extron-input-rescue #PWR0101
 U 1 1 5C74F12A
 P 5450 2550
@@
 	6200 2400 6250 2400
 $Comp
-L extron-input-rescue:C_Small-Device-extron-input-rescue C1
+L extron-input-rescue:C_Small-Device-extron-input-rescue-extron-input-rescue C1
 U 1 1 5C74F422
 P 5800 2300
@@
 	5900 2300 6250 2300
 $Comp
-L extron-input-rescue:GND-power-extron-input-rescue #PWR0102
+L extron-input-rescue:GND-power-extron-input-rescue-extron-input-rescue #PWR0102
 U 1 1 5C74FB45
 P 6750 2700
@@
 $EndComp
 $Comp
-L extron-input-rescue:SW_DPDT_x2-Switch-extron-input-rescue SW1
+L extron-input-rescue:SW_DPDT_x2-Switch-extron-input-rescue-extron-input-rescue SW1
 U 2 1 5C75001B
 P 5100 3400
@@
 $EndComp
 $Comp
-L extron-input-rescue:SW_DPDT_x2-Switch-extron-input-rescue SW1
+L extron-input-rescue:SW_DPDT_x2-Switch-extron-input-rescue-extron-input-rescue SW1
 U 1 1 5C7500A7
 P 5050 2200
@@
 NoConn ~ 2400 6200
 $Comp
-L extron-input-rescue:Conn_01x01-Connector_Generic-extron-input-rescue J8
+L extron-input-rescue:Conn_01x01-Connector_Generic-extron-input-rescue-extron-input-rescue J8
 U 1 1 5C7605B3
 P 2600 5600
@@
 $EndComp
 $Comp
-L extron-input-rescue:Conn_01x01-Connector_Generic-extron-input-rescue J9
+L extron-input-rescue:Conn_01x01-Connector_Generic-extron-input-rescue-extron-input-rescue J9
 U 1 1 5C76074F
 P 2600 5800
@@
 $EndComp
 $Comp
-L extron-input-rescue:Conn_01x01-Connector_Generic-extron-input-rescue J10
+L extron-input-rescue:Conn_01x01-Connector_Generic-extron-input-rescue-extron-input-rescue J10
 U 1 1 5C760785
 P 2600 6000
@@
 $EndComp
 $Comp
-L extron-input-rescue:Conn_01x01-Connector_Generic-extron-input-rescue J11
+L extron-input-rescue:Conn_01x01-Connector_Generic-extron-input-rescue-extron-input-rescue J11
 U 1 1 5C7607B9
 P 2600 6200
@@
 	5550 5700 5500 5700
 $Comp
-L extron-input-rescue:D_ALT-Device-extron-input-rescue D1
+L extron-input-rescue:D_ALT-Device-extron-input-rescue-extron-input-rescue D1
 U 1 1 5C84733C
 P 4350 5700
@@
 $EndComp
 $Comp
-L extron-input-rescue:R_US-Device-extron-input-rescue R2
+L extron-input-rescue:R_US-Device-extron-input-rescue-extron-input-rescue R2
 U 1 1 5C847B71
 P 4800 5700
@@
 $EndComp
 $Comp
-L extron-input-rescue:D_Zener-Device-extron-input-rescue D2
+L extron-input-rescue:D_Zener-Device-extron-input-rescue-extron-input-rescue D2
 U 1 1 5C847C9D
 P 5050 5850
@@
 SENSE
 $Comp
-L extron-input-rescue:GND-power-extron-input-rescue #PWR0103
+L extron-input-rescue:GND-power-extron-input-rescue-extron-input-rescue #PWR0103
 U 1 1 5C849937
 P 5050 6050
@@
 	5050 6000 5050 6050
 $Comp
-L extron-input-rescue:R_US-Device-extron-input-rescue R3
+L extron-input-rescue:R_US-Device-extron-input-rescue-extron-input-rescue R3
 U 1 1 5C84AF3E
 P 5350 5700
@@
 	4500 5700 4650 5700
 $Comp
-L extron-input-rescue:Conn_Coaxial-Connector-extron-input-rescue J2
+L extron-input-rescue:Conn_Coaxial-Connector-extron-input-rescue-extron-input-rescue J2
 U 1 1 5C8498CA
 P 8250 2050
@@
 $EndComp
 $Comp
-L extron-input-rescue:Conn_Coaxial-Connector-extron-input-rescue J3
+L extron-input-rescue:Conn_Coaxial-Connector-extron-input-rescue-extron-input-rescue J3
 U 1 1 5C849928
 P 8250 2900
@@
 $EndComp
 $Comp
-L extron-input-rescue:Conn_Coaxial-Connector-extron-input-rescue J4
+L extron-input-rescue:Conn_Coaxial-Connector-extron-input-rescue-extron-input-rescue J4
 U 1 1 5C84997A
 P 8250 3750
@@
 $EndComp
 $Comp
-L extron-input-rescue:Conn_Coaxial-Connector-extron-input-rescue J5
+L extron-input-rescue:Conn_Coaxial-Connector-extron-input-rescue-extron-input-rescue J5
 U 1 1 5C8499F8
 P 8250 4550

Commit message: Version 2.2 of extron input (move sense to top)
This revision moves the sense circuit to the top of the board, which
makes the audio plug a lot easier to get at, and you can throw your
esp32-switcher on the top of your extron.

Also cleaned up rescue files for eeschema. Come on, eeschema. Get your
shit together.
Parts:
- C1, C2: symbol extron-input-rescue:C_Small-Device-extron-input-rescue-extron-input-rescue -> Device:C_Small
- D1: symbol extron-input-rescue:D_ALT-Device-extron-input-rescue-extron-input-rescue -> Device:D_ALT
- D2: symbol extron-input-rescue:D_Zener-Device-extron-input-rescue-extron-input-rescue -> Device:D_Zener
- J1: symbol extron-input-rescue:SCART-F-Connector-extron-input-rescue-extron-input-rescue -> Connector:SCART-F
- J10, J11, J8, J9: symbol extron-input-rescue:Conn_01x01-Connector_Generic-extron-input-rescue-extron-input-rescue -> Connector_Generic:Conn_01x01
- J2, J3, J4, J5: symbol extron-input-rescue:Conn_Coaxial-Connector-extron-input-rescue-extron-input-rescue -> Connector:Conn_Coaxial
- J6: symbol extron-input-rescue:Conn_01x03_Male-Connector-extron-input-rescue-extron-input-rescue -> Connector:Conn_01x03_Male
- J7: symbol extron-input-rescue:Conn_01x02_Male-Connector-extron-input-rescue-extron-input-rescue -> Connector:Conn_01x02_Male
- R1, R2, R3: symbol extron-input-rescue:R_US-Device-extron-input-rescue-extron-input-rescue -> Device:R_US
- SW1: symbol extron-input-rescue:SW_DPDT_x2-Switch-extron-input-rescue-extron-input-rescue -> Switch:SW_DPDT_x2
- U1: symbol extron-input-rescue:LM1881-Video-extron-input-rescue-extron-input-rescue -> Video:LM1881
Changed lines of the file:
@@
 Sheet 1 1
 Title "Extron Scart Adapter (Input)"
-Date "2019-03-28"
-Rev "2.1"
+Date "2019-05-21"
+Rev "2.2"
 Comp "Rattboi (Bradon Kanyid)"
 Comment1 ""
@@
 GND
 $Comp
-L extron-input-rescue:SCART-F-Connector-extron-input-rescue-extron-input-rescue J1
+L Connector:SCART-F J1
 U 1 1 5C652397
 P 3850 3100
@@
 $EndComp
 $Comp
-L extron-input-rescue:Conn_01x03_Male-Connector-extron-input-rescue-extron-input-rescue J6
+L Connector:Conn_01x03_Male J6
 U 1 1 5C652866
 P 4650 4750
@@
 $EndComp
 $Comp
-L extron-input-rescue:Conn_01x02_Male-Connector-extron-input-rescue-extron-input-rescue J7
+L Connector:Conn_01x02_Male J7
 U 1 1 5C74DAFA
 P 5750 5800
@@
 $EndComp
 $Comp
-L extron-input-rescue:LM1881-Video-extron-input-rescue-extron-input-rescue U1
+L Video:LM1881 U1
 U 1 1 5C74DDC8
 P 6750 2400
@@
 $EndComp
 $Comp
-L extron-input-rescue:R_US-Device-extron-input-rescue-extron-input-rescue R1
+L Device:R_US R1
 U 1 1 5C74E55F
 P 5800 2850
@@
 $EndComp
 $Comp
-L extron-input-rescue:C_Small-Device-extron-input-rescue-extron-input-rescue C2
+L Device:C_Small C2
 U 1 1 5C74EC46
 P 5800 2500
@@
 	6000 2500 6200 2500
 $Comp
-L extron-input-rescue:GND-power-extron-input-rescue-extron-input-rescue #PWR0101
+L power:GND #PWR0101
 U 1 1 5C74F12A
 P 5450 2550
@@
 	6200 2400 6250 2400
 $Comp
-L extron-input-rescue:C_Small-Device-extron-input-rescue-extron-input-rescue C1
+L Device:C_Small C1
 U 1 1 5C74F422
 P 5800 2300
@@
 	5900 2300 6250 2300
 $Comp
-L extron-input-rescue:GND-power-extron-input-rescue-extron-input-rescue #PWR0102
+L power:GND #PWR0102
 U 1 1 5C74FB45
 P 6750 2700
@@
 $EndComp
 $Comp
-L extron-input-rescue:SW_DPDT_x2-Switch-extron-input-rescue-extron-input-rescue SW1
-U 2 1 5C75001B
-P 5100 3400
-F 0 "SW1" H 5100 3685 50  0000 C CNN
-F 1 "SW_DPDT_x2" H 5100 3594 50  0000 C CNN
-F 2 "Button_Switch_THT:SW_CuK_JS202011AQN_DPDT_Angled" H 5100 3400 50  0001 C CNN
-F 3 "" H 5100 3400 50  0001 C CNN
-F 4 "https://lcsc.com/product-detail/Toggle-Switches_C-K_JS202011AQN_C-K-JS202011AQN_C221662.html" H 5100 3400 50  0001 C CNN "Vendor"
-	2    5100 3400
-	1    0    0    -1
-$EndComp
-$Comp
-L extron-input-rescue:SW_DPDT_x2-Switch-extron-input-rescue-extron-input-rescue SW1
+L Switch:SW_DPDT_x2 SW1
 U 1 1 5C7500A7
 P 5050 2200
@@
 NoConn ~ 2400 6200
 $Comp
-L extron-input-rescue:Conn_01x01-Connector_Generic-extron-input-rescue-extron-input-rescue J8
+L Connector_Generic:Conn_01x01 J8
 U 1 1 5C7605B3
 P 2600 5600
@@
 $EndComp
 $Comp
-L extron-input-rescue:Conn_01x01-Connector_Generic-extron-input-rescue-extron-input-rescue J9
+L Connector_Generic:Conn_01x01 J9
 U 1 1 5C76074F
 P 2600 5800
@@
 $EndComp
 $Comp
-L extron-input-rescue:Conn_01x01-Connector_Generic-extron-input-rescue-extron-input-rescue J10
+L Connector_Generic:Conn_01x01 J10
 U 1 1 5C760785
 P 2600 6000
@@
 $EndComp
 $Comp
-L extron-input-rescue:Conn_01x01-Connector_Generic-extron-input-rescue-extron-input-rescue J11
+L Connector_Generic:Conn_01x01 J11
 U 1 1 5C7607B9
 P 2600 6200
@@
 	5550 5700 5500 5700
 $Comp
-L extron-input-rescue:D_ALT-Device-extron-input-rescue-extron-input-rescue D1
+L Device:D_ALT D1
 U 1 1 5C84733C
 P 4350 5700
@@
 $EndComp
 $Comp
-L extron-input-rescue:R_US-Device-extron-input-rescue-extron-input-rescue R2
+L Device:R_US R2
 U 1 1 5C847B71
 P 4800 5700
@@
 $EndComp
 $Comp
-L extron-input-rescue:D_Zener-Device-extron-input-rescue-extron-input-rescue D2
+L Device:D_Zener D2
 U 1 1 5C847C9D
 P 5050 5850
@@
 SENSE
 $Comp
-L extron-input-rescue:GND-power-extron-input-rescue-extron-input-rescue #PWR0103
+L power:GND #PWR0103
 U 1 1 5C849937
 P 5050 6050
@@
 	5050 6000 5050 6050
 $Comp
-L extron-input-rescue:R_US-Device-extron-input-rescue-extron-input-rescue R3
+L Device:R_US R3
 U 1 1 5C84AF3E
 P 5350 5700
@@
 	4500 5700 4650 5700
 $Comp
-L extron-input-rescue:Conn_Coaxial-Connector-extron-input-rescue-extron-input-rescue J2
+L Connector:Conn_Coaxial J2
 U 1 1 5C8498CA
 P 8250 2050
@@
 $EndComp
 $Comp
-L extron-input-rescue:Conn_Coaxial-Connector-extron-input-rescue-extron-input-rescue J3
+L Connector:Conn_Coaxial J3
 U 1 1 5C849928
 P 8250 2900
@@
 $EndComp
 $Comp
-L extron-input-rescue:Conn_Coaxial-Connector-extron-input-rescue-extron-input-rescue J4
+L Connector:Conn_Coaxial J4
 U 1 1 5C84997A
 P 8250 3750
@@
 $EndComp
 $Comp
-L extron-input-rescue:Conn_Coaxial-Connector-extron-input-rescue-extron-input-rescue J5
+L Connector:Conn_Coaxial J5
 U 1 1 5C8499F8
 P 8250 4550
@@
 Wire Wire Line
 	5250 3800 5250 4750
+$Comp
+L Switch:SW_DPDT_x2 SW1
+U 2 1 5C75001B
+P 5100 3400
+F 0 "SW1" H 5100 3685 50  0000 C CNN
+F 1 "SW_DPDT_x2" H 5100 3594 50  0000 C CNN
+F 2 "Button_Switch_THT:SW_CuK_JS202011AQN_DPDT_Angled" H 5100 3400 50  0001 C CNN
+F 3 "" H 5100 3400 50  0001 C CNN
+F 4 "https://lcsc.com/product-detail/Toggle-Switches_C-K_JS202011AQN_C-K-JS202011AQN_C221662.html" H 5100 3400 50  0001 C CNN "Vendor"
+	2    5100 3400
+	1    0    0    -1
+$EndComp
 $EndSCHEMATC
